Commit message: new features

File: denis_v1_description/urdf/camera.xacro (robot description, xacro)
@@ -1,9 +1,12 @@
 <?xml version="1.0"?>
 <robot xmlns:xacro="http://www.ros.org/wiki/xacro">
+    <xacro:property name="camera_length" value="0.03" />
+    <xacro:property name="camera_width" value="${base_width / 3}" />
+    <xacro:property name="camera_height" value="${base_height / 3}" />
     <xacro:include filename="inertia.xacro" />
     <link name="camera_link">
         <visual>
             <geometry>
-                <box size="0.1 ${base_width / 3} ${base_height / 3}" />
+                <box size="${camera_length} ${camera_width} ${camera_height}" />
             </geometry>
             <origin xyz="0 0 0" rpy="0 0 0" />
@@ -12,9 +15,9 @@
         <collision>
             <geometry>
-                <box size="0.1 ${base_width / 3} ${base_height / 3}" />
+                <box size="${camera_length} ${camera_width} ${camera_height}" />
             </geometry>
             <origin xyz="0 0 0" rpy="0 0 0" />
         </collision>
-        <xacro:box_inertia m="0.1" w="${base_width / 3}" h="${base_height / 3}" d="0.1"
+        <xacro:box_inertia m="0.1" x="${camera_length}" y="${camera_width}" z="${camera_height}"
             o_xyz="0 0 0" o_rpy="0 0 0" />
     </link>
@@ -22,20 +25,16 @@
         <parent link="base_link" />
         <child link="camera_link" />
-        <origin xyz="${base_length / 2} 0 ${base_height / 2}" rpy="0 0 0" />
+        <origin xyz="${base_length / 2.0 + camera_length / 2.0} 0 ${base_height / 2.0}" rpy="0 0 0" />
     </joint>
-    <link name="camera_depth_frame" />
+    <link name="camera_link_optical" />
     <joint name="camera_depth_joint" type="fixed">
         <origin xyz="0 0 0" rpy="${-pi/2} 0 ${-pi/2}" />
         <parent link="camera_link" />
-        <child link="camera_depth_frame" />
+        <child link="camera_link_optical" />
     </joint>
-    <gazebo reference="camera_depth_frame">
-        <sensor name="depth_camera" type="rgbd_camera">
-            <gz_frame_id>camera_depth_frame</gz_frame_id>
-            <visualize>true</visualize>
-            <update_rate>30.0</update_rate>
-            <topic>/depth_camera</topic>
-            <camera name="camera">
-                <horizontal_fov>1.047198</horizontal_fov>
+    <gazebo reference="camera_link">
+        <sensor name="camera" type="camera">
+            <camera>
+                <horizontal_fov>1.3962634</horizontal_fov>
                 <image>
                     <width>640</width>
@@ -44,8 +43,19 @@
                 </image>
                 <clip>
-                    <near>0.05</near>
-                    <far>3</far>
+                    <near>0.1</near>
+                    <far>15</far>
                 </clip>
+                <noise>
+                    <type>gaussian</type>
+                    <mean>0.0</mean>
+                    <stddev>0.007</stddev>
+                </noise>
+                <optical_frame_id>camera_link_optical</optical_frame_id>
+                <camera_info_topic>camera/camera_info</camera_info_topic>
             </camera>
+            <always_on>1</always_on>
+            <update_rate>20</update_rate>
+            <visualize>true</visualize>
+            <topic>camera/image_raw</topic>
         </sensor>
     </gazebo>

File: denis_v1_description/urdf/common_properties.xacro (robot description, xacro)
@@ -10,11 +10,3 @@
         <color rgba="1 ${165/255} 0 1" />
     </material>
-    <xacro:property name="base_length" value="0.6" />
-    <xacro:property name="base_width" value="0.4" />
-    <xacro:property name="base_height" value="0.2" />
-    <xacro:property name="lidar_radius" value="0.1" />
-    <xacro:property name="lidar_length" value="0.04" />
-    <xacro:property name="wheel_radius" value="0.1" />
-    <xacro:property name="wheel_length" value="0.05" />
-    <xacro:property name="sphere_front_radius" value="0.05" />
 </robot>

File: denis_v1_description/urdf/denis.urdf.xacro (robot description, xacro)
@@ -1,8 +1,8 @@
-<?xml version="1.0" ?>
-<robot name="denis_v1" xmlns:xacro="http://www.ros.org/wiki/xacro">
+<?xml version="1.0"?>
+<robot name="denis" xmlns:xacro="http://www.ros.org/wiki/xacro">
     <xacro:include filename="common_properties.xacro" />
     <xacro:include filename="mobile_base.xacro" />
-    <xacro:include filename="mobile_base.ros2_control.xacro"/>
-    <xacro:include filename="lidar.xacro"/>
+    <xacro:include filename="lidar.xacro" />
     <xacro:include filename="camera.xacro" />
+    <xacro:include filename="mobile_base_gazebo.xacro" />
 </robot>

File: denis_v1_description/urdf/inertia.xacro (robot description, xacro)
@@ -22,10 +22,14 @@
         </inertial>
     </xacro:macro>
-    <xacro:macro name="box_inertia" params="m w h d o_xyz o_rpy">
+    <xacro:macro name="box_inertia" params="m x y z o_xyz o_rpy">
         <inertial>
             <origin xyz="${o_xyz}" rpy="${o_rpy}" />
             <mass value="${m}" />
-            <inertia ixx="${(m/12) * (h*h + d*d)}" ixy="0.0" ixz="0.0" iyy="${(m/12) * (w*w + d*d)}"
-                iyz="0.0" izz="${(m/12) * (w*w + h*h)}" />
+            <inertia
+                ixx="${(m/12) * (y*y + z*z)}"
+                ixy="0.0" ixz="0.0"
+                iyy="${(m/12) * (x*x + z*z)}"
+                iyz="0.0"
+                izz="${(m/12) * (x*x + y*y)}" />
         </inertial>
     </xacro:macro>

File: denis_v1_description/urdf/lidar.xacro (robot description, xacro)
@@ -1,4 +1,6 @@
 <?xml version="1.0"?>
 <robot xmlns:xacro="http://www.ros.org/wiki/xacro">
+    <xacro:property name="lidar_radius" value="0.1" />
+    <xacro:property name="lidar_length" value="0.04" />
     <link name="lidar_link">
         <visual>

File: denis_v1_description/urdf/mobile_base.xacro (robot description, xacro)
@@ -1,4 +1,10 @@
 <?xml version="1.0"?>
 <robot xmlns:xacro="http://www.ros.org/wiki/xacro">
+    <xacro:property name="base_length" value="0.6" />
+    <xacro:property name="base_width" value="0.4" />
+    <xacro:property name="base_height" value="0.2" />
+    <xacro:property name="wheel_radius" value="0.1" />
+    <xacro:property name="wheel_length" value="0.05" />
+    <xacro:property name="sphere_front_radius" value="0.05" />
     <xacro:include filename="inertia.xacro" />
     <link name="base_footprint" />
@@ -17,5 +23,6 @@
             <origin xyz="0 0 ${base_height/2}" rpy="0 0 0" />
         </collision>
-        <xacro:box_inertia m="5" w="${base_width}" h="${base_height}" d="${base_length}" o_xyz="0 0 ${base_height/2}" o_rpy="0 0 0" />
+        <xacro:box_inertia m="5" x="${base_length}" y="${base_width}" z="${base_height}"
+            o_xyz="0 0 ${base_height/2}" o_rpy="0 0 0" />
     </link>
     <link name="left_wheel_link">
