Commit message: simulation fixes

File: denis_v1_description/urdf/gazebo_control.xacro (robot description, xacro)
@@ -1,8 +1,4 @@
 <?xml version="1.0"?>
 <robot xmlns:xacro="http://www.ros.org/wiki/xacro">
-    <gazebo reference="caster_wheel_link">
-        <mu1 value="0.1" />
-        <mu2 value="0.1" />
-    </gazebo>
     <gazebo>
         <plugin

File: denis_v1_description/urdf/lidar.xacro (robot description, xacro)
@@ -1,6 +1,6 @@
 <?xml version="1.0"?>
 <robot xmlns:xacro="http://www.ros.org/wiki/xacro">
-    <xacro:property name="lidar_radius" value="0.1" />
-    <xacro:property name="lidar_length" value="0.04" />
+    <xacro:property name="lidar_radius" value="0.035" />
+    <xacro:property name="lidar_length" value="0.03" />
     <link name="lidar_link">
         <visual>
@@ -23,5 +23,5 @@
         <parent link="base_link" />
         <child link="lidar_link" />
-        <origin xyz="0 0 ${base_height + lidar_length/2.0}" rpy="0 0 0" />
+        <origin xyz="-${base_length/8} 0 ${base_height + lidar_length/2.0}" rpy="0 0 0" />
     </joint>
     <gazebo reference="lidar_link">

File: denis_v1_description/urdf/mobile_base.xacro (robot description, xacro)
@@ -1,10 +1,10 @@
 <?xml version="1.0"?>
 <robot xmlns:xacro="http://www.ros.org/wiki/xacro">
-    <xacro:property name="base_length" value="0.6" />
-    <xacro:property name="base_width" value="0.4" />
+    <xacro:property name="base_length" value="0.345" />
+    <xacro:property name="base_width" value="0.231" />
     <xacro:property name="base_height" value="0.2" />
-    <xacro:property name="wheel_radius" value="0.1" />
-    <xacro:property name="wheel_length" value="0.05" />
-    <xacro:property name="sphere_front_radius" value="0.05" />
+    <xacro:property name="wheel_radius" value="0.0325" />
+    <xacro:property name="wheel_length" value="0.027" />
+    <xacro:property name="sphere_front_radius" value="${wheel_radius/2}" />
     <xacro:include filename="inertia.xacro" />
     <link name="base_footprint" />
@@ -40,5 +40,5 @@
             <origin xyz="0 0 0" rpy="${pi / 2.0} 0 0" />
         </collision>
-        <xacro:cylinder_inertia m="1" radius="${wheel_radius}"
+        <xacro:cylinder_inertia m="0.010" radius="${wheel_radius}"
             length="${wheel_length}" o_xyz="0 0 0" o_rpy="${pi / 2.0} 0 0" />
     </link>
@@ -59,5 +59,5 @@
             <origin xyz="0 0 0" rpy="${pi / 2.0} 0 0" />
         </collision>
-        <xacro:cylinder_inertia m="1" radius="${wheel_radius}"
+        <xacro:cylinder_inertia m="0.010" radius="${wheel_radius}"
             length="${wheel_length}" o_xyz="0 0 0" o_rpy="${pi / 2.0} 0 0" />
     </link>
@@ -76,5 +76,5 @@
             <origin xyz="0 0 0" rpy="0 0 0" />
         </collision>
-        <xacro:sphere_inertia m="0.5" r="${sphere_front_radius}" o_xyz="0 0 0" o_rpy="0 0 0" />
+        <xacro:sphere_inertia m="0.010" r="${sphere_front_radius}" o_xyz="0 0 0" o_rpy="0 0 0" />
     </link>
     <joint name="base_footprint_base_joint" type="fixed">
@@ -100,3 +100,7 @@
         <axis xyz="0 1 0" />
     </joint>
+    <gazebo reference="caster_wheel_link">
+        <mu1 value="0.001"/>
+        <mu2 value="0.001"/>
+    </gazebo>
 </robot>

File: denis_v1_description/urdf/ros2_control.xacro (robot description, xacro)
@@ -56,6 +56,6 @@
     <gazebo>
     <plugin name="gz_ros2_control::GazeboSimROS2ControlPlugin" filename="libgz_ros2_control-system.so">
+        <parameters>$(find denis_v1_bringup)/config/gazebo_control_use_sim.yaml</parameters>
         <parameters>$(find denis_v1_bringup)/config/denis_controllers.yaml</parameters>
-        <parameters>$(find denis_v1_bringup)/config/gazebo_control_use_sim.yaml</parameters>
     </plugin>
 </gazebo>
