Commit message: small changes on shape

File: denis_v1_description/urdf/mobile_base.xacro (robot description, xacro)
@@ -1,6 +1,6 @@
 <?xml version="1.0"?>
 <robot xmlns:xacro="http://www.ros.org/wiki/xacro">
-    <xacro:property name="base_length" value="0.345" />
-    <xacro:property name="base_width" value="0.24" />
+    <xacro:property name="base_length" value="0.36" />
+    <xacro:property name="base_width" value="0.245" />
     <xacro:property name="base_height" value="0.2" />
     <xacro:property name="wheel_radius" value="0.0325" />
