Commit message: fixes

File: denis_v1_description/ros2_control/ros2_control.xacro (robot description, xacro)
@@ -5,25 +5,23 @@
             <hardware>
                 <plugin>denis_diff_hardware/DiffDenisSystemHardware</plugin>
-                <param name="left_wheel_name">left_wheel_joint</param>
-                <param name="right_wheel_name">right_wheel_joint</param>
+                <param name="left_wheel_name">base_left_wheel_joint</param>
+                <param name="right_wheel_name">base_right_wheel_joint</param>
                 <param name="loop_rate">30</param>
-                <param name="device">/dev/ttyUSB0</param>
-                <param name="baud_rate">115200</param>
+                <param name="device">/dev/serial/by-id/usb-1a86_USB_Serial-if00-port0</param>
+                <param name="baud_rate">57600</param>
                 <param name="timeout_ms">1000</param>
                 <param name="enc_counts_per_rev">660</param>
+                <param name="pid_p">20</param>
+                <param name="pid_d">12</param>
+                <param name="pid_i">0</param>
+                <param name="pid_o">50</param>
             </hardware>
             <joint name="base_left_wheel_joint">
-                <command_interface name="velocity">
-                    <param name="min">-10</param>
-                    <param name="max">10</param>
-                </command_interface>
+                <command_interface name="velocity" />
                 <state_interface name="position" />
                 <state_interface name="velocity" />
             </joint>
             <joint name="base_right_wheel_joint">
-                <command_interface name="velocity">
-                    <param name="min">-10</param>
-                    <param name="max">10</param>
-                </command_interface>
+                <command_interface name="velocity" />
                 <state_interface name="position" />
                 <state_interface name="velocity" />

File: denis_v1_description/urdf/mobile_base.xacro (robot description, xacro)
@@ -2,5 +2,5 @@
 <robot xmlns:xacro="http://www.ros.org/wiki/xacro">
     <xacro:property name="base_length" value="0.345" />
-    <xacro:property name="base_width" value="0.231" />
+    <xacro:property name="base_width" value="0.24" />
     <xacro:property name="base_height" value="0.2" />
     <xacro:property name="wheel_radius" value="0.0325" />

Commit message: navigation-slam-works fine

File: denis_v1_description/ros2_control/ros2_control.xacro (robot description, xacro)
@@ -11,7 +11,7 @@
                 <param name="baud_rate">57600</param>
                 <param name="timeout_ms">1000</param>
-                <param name="enc_counts_per_rev">660</param>
-                <param name="pid_p">20</param>
-                <param name="pid_d">12</param>
+                <param name="enc_counts_per_rev">1320</param>
+                <param name="pid_p">25</param>
+                <param name="pid_d">5</param>
                 <param name="pid_i">0</param>
                 <param name="pid_o">50</param>

File: denis_v1_description/urdf/mobile_base.xacro (robot description, xacro)
@@ -4,6 +4,6 @@
     <xacro:property name="base_width" value="0.245" />
     <xacro:property name="base_height" value="0.2" />
-    <xacro:property name="wheel_radius" value="0.0325" />
-    <xacro:property name="wheel_length" value="0.027" />
+    <xacro:property name="wheel_radius" value="0.03" />
+    <xacro:property name="wheel_length" value="0.026" />
     <xacro:property name="sphere_front_radius" value="${wheel_radius/2}" />
     <xacro:include filename="inertia.xacro" />
@@ -91,5 +91,5 @@
         <parent link="base_link" />
         <child link="left_wheel_link" />
-        <origin xyz="-${base_length/3} ${base_width/2 + wheel_length/2} 0" rpy="0 0 0" />
+        <origin xyz="-${base_length/3} ${base_width/2 + wheel_length/2 + 0.009} 0" rpy="0 0 0" />
         <axis xyz="0 1 0" />
     </joint>
@@ -97,5 +97,5 @@
         <parent link="base_link" />
         <child link="right_wheel_link" />
-        <origin xyz="-${base_length/3} -${base_width/2 + wheel_length/2} 0" rpy="0 0 0" />
+        <origin xyz="-${base_length/3} -${base_width/2 + wheel_length/2  + 0.009} 0" rpy="0 0 0" />
         <axis xyz="0 1 0" />
     </joint>
